File: Hardware/SED Ethernet/sed_ethernet.brd (EAGLE design)
At the start: 50 x 23.8 mm, 30 parts, among them IC1 ENC28J60SSOP, Q2 25MHz

Commit message: Cristal con toma de tierra
Parts:
- Q2: device SparkFun:CRYSTAL-SMD-5X3 -> sed_library:CRYSTAL-SMD-5X3
- moved C20 2.17 mm to (19.2, 20.3), turned to 90 degrees
- moved R8 2.16 mm to (15.4, 18.0)
Connections:
- net GND: now also Q2.2, Q2.4
Routing:
- net GND: track 151.8 -> 159.3 mm, vias 1 -> 3
- net N$9: track 33.2 -> 36.9 mm
- net N$7: track 4.37 -> 6.64 mm
- net N$23: track 9.38 -> 11.4 mm
- net N$13: track 46.4 -> 47.2 mm
